File: mainboard/esp32-watch.sch (EAGLE design)
At the start: 15 parts, among them J1 CON-MOLEX_0532610671, U1 ESP-WROOM-32

Commit message: started to add NRF24L01 header
Parts:
- added U$1: NRF24L01, VanEagleLib:NRF24L01
Connections:
- net 3V3: now also U$1.3.3V
- net GND: now also U$1.GND
- net IO18: now also U$1.MISO
- net IO19: now also U$1.SCK
- net IO21: now also U$1.MOSI
Changed lines of the file:
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@@
 <part name="P+1" library="supply1" deviceset="+5V" device=""/>
 <part name="+3V1" library="supply1" deviceset="+3V3" device=""/>
+<part name="U$1" library="VanEagleLib" library_urn="urn:adsk.eagle:library:5408729" deviceset="NRF24L01" device=""/>
+<part name="GND7" library="supply1" deviceset="GND" device=""/>
 </parts>
 <sheets>
@@
 <instance part="P+1" gate="1" x="15.24" y="53.34"/>
 <instance part="+3V1" gate="G$1" x="86.36" y="50.8"/>
+<instance part="U$1" gate="G$1" x="139.7" y="40.64"/>
+<instance part="GND7" gate="1" x="101.6" y="43.18"/>
 </instances>
 <busses>
@@
 <label x="236.22" y="160.02" size="1.778" layer="95"/>
 </segment>
+<segment>
+<pinref part="U$1" gate="G$1" pin="MOSI"/>
+<wire x1="154.94" y1="40.64" x2="160.02" y2="40.64" width="0.1524" layer="91"/>
+<label x="160.02" y="40.64" size="1.778" layer="95"/>
+</segment>
 </net>
 <net name="IO19" class="0">
@@
 <label x="134.62" y="78.74" size="1.778" layer="95"/>
 </segment>
+<segment>
+<pinref part="U$1" gate="G$1" pin="SCK"/>
+<wire x1="121.92" y1="40.64" x2="111.76" y2="40.64" width="0.1524" layer="91"/>
+<label x="111.76" y="40.64" size="1.778" layer="95"/>
+</segment>
 </net>
 <net name="IO18" class="0">
@@
 <wire x1="121.92" y1="81.28" x2="139.7" y2="81.28" width="0.1524" layer="91"/>
 <label x="134.62" y="81.28" size="1.778" layer="95"/>
+</segment>
+<segment>
+<pinref part="U$1" gate="G$1" pin="MISO"/>
+<wire x1="121.92" y1="38.1" x2="111.76" y2="38.1" width="0.1524" layer="91"/>
+<label x="111.76" y="38.1" size="1.778" layer="95"/>
 </segment>
 </net>
@@
 <wire x1="96.52" y1="86.36" x2="81.28" y2="86.36" width="0.1524" layer="91"/>
 <label x="81.28" y="86.36" size="1.778" layer="95"/>
+</segment>
+<segment>
+<pinref part="U$1" gate="G$1" pin="3.3V"/>
+<wire x1="154.94" y1="45.72" x2="160.02" y2="45.72" width="0.1524" layer="91"/>
+<label x="160.02" y="45.72" size="1.778" layer="95"/>
 </segment>
 </net>
@@
 <wire x1="22.86" y1="17.78" x2="22.86" y2="25.4" width="0.1524" layer="91"/>
 </segment>
-</net>
+<segment>
+<pinref part="U$1" gate="G$1" pin="GND"/>
+<wire x1="121.92" y1="45.72" x2="116.84" y2="45.72" width="0.1524" layer="91"/>
+<wire x1="116.84" y1="45.72" x2="101.6" y2="45.72" width="0.1524" layer="91"/>
+<pinref part="GND7" gate="1" pin="GND"/>
+</segment>
+</net>
